File: ExpansionBoard/sfg_adapter.brd (EAGLE design)
At the start: 116 x 41 mm, 7 parts, among them X1 SFGSFG, X2 SFG_CABLESFG_CABLE, X3 RCA, X4 RCA, X5 SFG-20, X6 MIDI_CONN_FEMALE_SUPPORT, X7 MIDI_CONN_FEMALE_SUPPORT

Commit message: New board revision
New board revision + Gerbers
Routing:
- net N$2: track 0.00 -> 10.9 mm
- net N$1: track 0.00 -> 10.9 mm
Other:
- board text added: "GND"
Changed lines of the file:
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@@
 <setting verticaltext="up"/>
 </settings>
-<grid distance="0.2" unitdist="mm" unit="mm" style="lines" multiple="1" display="yes" altdistance="1" altunitdist="mm" altunit="mm"/>
+<grid distance="0.1" unitdist="mm" unit="mm" style="lines" multiple="1" display="yes" altdistance="1" altunitdist="mm" altunit="mm"/>
 <layers>
 <layer number="1" name="Top" color="4" fill="1" visible="yes" active="yes"/>
@@
 <wire x1="107" y1="145" x2="76" y2="145" width="0.2" layer="26"/>
 <wire x1="76" y1="145" x2="76" y2="151.5" width="0.2" layer="26"/>
+<circle x="23" y="145.5" radius="1.0816625" width="0.4064" layer="16"/>
+<circle x="8" y="145.5" radius="1.0630125" width="0.4064" layer="16"/>
+<text x="6.8" y="153.6" size="1" layer="25">GND</text>
+<text x="21.8" y="153.6" size="1" layer="25">GND</text>
+<circle x="23" y="145.5" radius="1.140175" width="0.5" layer="30"/>
+<circle x="8" y="145.5" radius="1.140175" width="0.5" layer="30"/>
 </plain>
 <attributes>
@@
 <wire x1="13.3" y1="144.1" x2="2.7" y2="144.1" width="0.5" layer="1"/>
 </signal>
+<signal name="N$1">
+<wire x1="13.3" y1="144.1" x2="8" y2="144.1" width="0.5" layer="16"/>
+<wire x1="2.7" y1="144.1" x2="8" y2="144.1" width="0.5" layer="16"/>
+<wire x1="8" y1="144.1" x2="8" y2="144.4" width="0.5" layer="16"/>
+</signal>
+<signal name="N$2">
+<wire x1="28.3" y1="144.1" x2="23" y2="144.1" width="0.5" layer="16"/>
+<wire x1="17.7" y1="144.1" x2="23" y2="144.1" width="0.5" layer="16"/>
+<wire x1="23" y1="144.1" x2="23" y2="144.4" width="0.5" layer="16"/>
+</signal>
 </signals>
